Commit message: feat(navigation): changed robot

File: urdf/robot.urdf (robot description, URDF)
Before this commit: robot differential_drive_rob, 6 links, 5 joints
Links:
- link link_chassis: geometry collision box size=0.4 0.25 0.12; visual box size=0.4 0.25 0.12
Joints:
- joint left_wheel_hinge_back: origin xyz=-0.2 0.30 0 rpy=0 0 0 -> xyz=-0.13 0.13 0 rpy=0 0 0
- joint left_wheel_hinge_front: origin xyz=0.2 0.30 0 rpy=0 0 0 -> xyz=0.13 0.13 0 rpy=0 0 0
- joint right_wheel_hinge_back: origin xyz=-0.2 -0.30 0 rpy=0 0 0 -> xyz=-0.13 -0.13 0 rpy=0 0 0
- joint right_wheel_hinge_front: origin xyz=0.2 -0.30 0 rpy=0 0 0 -> xyz=0.13 -0.13 0 rpy=0 0 0
